File: OC64.kicad_pcb (KiCad board)
At the start: 2 copper layers, 360.2 x 122.6 mm, 147 parts, among them SW1 SW_ESC, SW10 SW_9, SW11 SW_0, SW12 SW_-, SW13 SW_=, SW14 SW_BACK, SW15 SW_DEL, SW16 SW_F1, SW17 SW_TAB, SW18 SW_Q, SW19 SW_W, SW2 SW_1, SW20 SW_E, SW21 SW_R, SW22 SW_T, SW23 SW_Y, SW24 SW_U, SW25 SW_I, SW26 SW_O, SW27 SW_P, SW28 SW_[, SW29 SW_], SW3 SW_2, SW30 SW_\, SW31 SW_PGUP, SW32 SW_F2, SW33-1 SW_STPCAP, SW33-2 SW_CAPS, SW34 SW_A, SW35 SW_S, SW36 SW_D, SW37 SW_F, SW38 SW_G, SW39 SW_H, SW4 SW_3, SW40 SW_J, SW41 SW_K, SW42 SW_L, SW43 SW_;, SW44 SW_', SW45 SW_RET, SW46 SW_PGDN, SW47 SW_F3, SW48 SW_SHIFT, SW49 SW_Z, SW5 SW_4, SW50 SW_X, SW51 SW_C, SW52 SW_V, SW53 SW_B, SW54 SW_N, SW55 SW_M, SW56 SW_,, SW57 SW_., SW58 SW_/, SW59 SW_SHIFT, SW6 SW_5, SW60 SW_HOME, SW61 SW_END, SW62 SW_F4, SW63 SW_CTRL, SW64 SW_LSPAC, SW65-1 SW_SPACE, SW65-2 SW_RSPAC, SW66 SW_ALT, SW67-1 SW_META, SW67-2 SW_META, SW7 SW_6, SW8 SW_7, SW9 SW_8, U1 ProMicro

Commit message: Added led pin & a text
Parts:
- added D68: LED, Connector_PinHeader_2.54mm:PinHeader_1x02_P2.54mm_Vertical, B.Cu at (34.5, 70.5)
- added R1: 1k, Keebio-Parts:Resistor-Compact, B.Cu at (44.4, 70.5)
Routing:
- net VCC: track 0.00 -> 309.1 mm
- net GND: track 20.9 -> 0.00 mm, vias 0 -> 6
- net Net-(D68-Pad1): track 0.00 -> 5.92 mm
Other:
- board text added: "**** ORTHOLINEAR COMMODORE 64 BASIC V1 ****"
- board text added: "64K RAM SYSTEM 38911 BASIC BYTES FREE"
- board text added: "@"
- board text added: "IKNO OC64:~~$"
- board text added: "READY."
- board text added: "▮"

Commit message: updated header pin for the LED to be on the correct side
Parts:
- moved D68 329.2 mm to (363.7, 69.1)
- moved R1 313.4 mm to (357.8, 67.9), turned to 90 degrees
Routing:
- net VCC: track 309.1 -> 43.6 mm
- net Net-(D68-Pad1): track 5.92 -> 7.72 mm
Changed lines of the file:
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@@
   (general
     (thickness 1.6)
-    (drawings 18)
-    (tracks 373)
+    (drawings 24)
+    (tracks 377)
     (zones 0)
     (modules 149)
@@
       (drillshape 0)
       (scaleselection 1)
-      (outputdirectory ""))
+      (outputdirectory "gerbers/"))
   )
   (net 0 "")
@@
   )
   (module Connector_PinHeader_2.54mm:PinHeader_1x02_P2.54mm_Vertical (layer B.Cu)
-    (at 34.528096 70.544472)
+    (at 363.736243 69.056308)
     (descr "Through hole straight pin header, 1x02, 2.54mm pitch, single row")
     (tags "Through hole pin header THT 1x02 2.54mm single row")
@@
   )
   (module Keebio-Parts:Resistor-Compact (layer B.Cu)
-    (at 44.350744 70.544472)
+    (at 357.783113 67.865682 90)
     (attr smd)
-    (fp_text reference R1 (at 0 0) (layer F.SilkS)
+    (fp_text reference R1 (at 0 0 90) (layer F.SilkS)
       (effects (font (size 0.8 0.8) (thickness 0.15)))
     )
-    (fp_text value 1k (at 0 0) (layer B.SilkS)
+    (fp_text value 1k (at 0 0 90) (layer B.SilkS)
       (effects (font (size 0.8 0.8) (thickness 0.15)) (justify mirror))
     )
@@
     (fp_line (start -2.54 1.016) (end -2.286 1.016) (layer B.SilkS) (width 0.15))
     (fp_line (start -2.794 0.762) (end -2.54 1.016) (layer B.SilkS) (width 0.15))
-    (pad 2 thru_hole circle (at -3.9 0) (size 1.6 1.6) (drill 1) (layers *.Cu *.Mask B.SilkS)
+    (pad 2 thru_hole circle (at -3.9 0 90) (size 1.6 1.6) (drill 1) (layers *.Cu *.Mask B.SilkS)
       (net 90 "Net-(D68-Pad1)"))
-    (pad 1 thru_hole circle (at 3.9 0) (size 1.6 1.6) (drill 1) (layers *.Cu *.Mask)
+    (pad 1 thru_hole circle (at 3.9 0 90) (size 1.6 1.6) (drill 1) (layers *.Cu *.Mask)
       (net 80 GND))
   )
@@
       (net 69 "Net-(D63-Pad2)"))
   )
+  (gr_text "64K RAM SYSTEM  38911 BASIC BYTES FREE" (at 317.5 165.5) (layer B.SilkS)
+    (effects (font (size 1.5 1.5) (thickness 0.3)) (justify mirror))
+  )
+  (gr_text "IKNO  OC64:~~$ " (at 345.5 172.35) (layer B.SilkS)
+    (effects (font (size 1.5 1.5) (thickness 0.3)) (justify left mirror))
+  )
+  (gr_text @ (at 338.85 172.05) (layer B.SilkS)
+    (effects (font (size 2 2) (thickness 0.2)) (justify mirror))
+  )
+  (gr_text ▮ (at 327.5 172.1) (layer B.SilkS)
+    (effects (font (size 2 1.5) (thickness 0.3)) (justify mirror))
+  )
+  (gr_text READY. (at 345.5 169.5) (layer B.SilkS)
+    (effects (font (size 1.5 1.5) (thickness 0.3)) (justify left mirror))
+  )
+  (gr_text "**** ORTHOLINEAR COMMODORE 64 BASIC V1 ****" (at 317.301829 162.2) (layer B.SilkS)
+    (effects (font (size 1.5 1.5) (thickness 0.3)) (justify mirror))
+  )
   (gr_text ▮ (at 306.225 172.125) (layer F.SilkS)
     (effects (font (size 2 1.5) (thickness 0.3)))
@@
   (segment (start 333.254929 62.805416) (end 337.765965 67.316452) (width 0.25) (layer F.Cu) (net 83))
   (segment (start 332.052848 62.805416) (end 333.254929 62.805416) (width 0.25) (layer F.Cu) (net 83))
-  (segment (start 335.688365 84.173701) (end 336.564664 85.05) (width 0.25) (layer F.Cu) (net 84))
-  (segment (start 320.369135 68.854471) (end 335.688365 84.173701) (width 0.25) (layer F.Cu) (net 84))
-  (segment (start 35.378095 68.854471) (end 320.369135 68.854471) (width 0.25) (layer F.Cu) (net 84))
-  (segment (start 34.528096 68.004472) (end 35.378095 68.854471) (width 0.25) (layer F.Cu) (net 84))
+  (segment (start 363.736243 66.516308) (end 340.160662 66.516308) (width 0.25) (layer F.Cu) (net 84))
+  (segment (start 337.440963 84.173701) (end 336.564664 85.05) (width 0.25) (layer F.Cu) (net 84))
+  (segment (start 338.215975 83.398689) (end 337.440963 84.173701) (width 0.25) (layer F.Cu) (net 84))
+  (segment (start 338.215975 68.460995) (end 338.215975 83.398689) (width 0.25) (layer F.Cu) (net 84))
+  (segment (start 340.160662 66.516308) (end 338.215975 68.460995) (width 0.25) (layer F.Cu) (net 84))
   (segment (start 237.187072 155.152947) (end 227.164568 155.152947) (width 0.25) (layer F.Cu) (net 85) (status 10))
   (segment (start 227.164568 155.152947) (end 225.122064 157.195451) (width 0.25) (layer F.Cu) (net 85) (status 20))
@@
   (segment (start 134.79324 155.152703) (end 110.48324 155.152703) (width 0.25) (layer F.Cu) (net 89) (status 10))
   (segment (start 110.48324 155.152703) (end 108.44074 157.195203) (width 0.25) (layer F.Cu) (net 89) (status 20))
-  (segment (start 40.450744 70.544472) (end 34.528096 70.544472) (width 0.25) (layer F.Cu) (net 90))
+  (segment (start 358.914483 71.765682) (end 357.783113 71.765682) (width 0.25) (layer F.Cu) (net 90))
+  (segment (start 362.126869 71.765682) (end 358.914483 71.765682) (width 0.25) (layer F.Cu) (net 90))
+  (segment (start 363.736243 70.156308) (end 362.126869 71.765682) (width 0.25) (layer F.Cu) (net 90))
+  (segment (start 363.736243 69.056308) (end 363.736243 70.156308) (width 0.25) (layer F.Cu) (net 90))
   (zone (net 80) (net_name GND) (layer F.Cu) (hatch edge 0.508)
     (connect_pads (clearance 0.508))
